Commit message: test loam_velodyne on scout

File: packages/octomap_scout/urdf/scout_v2.xacro (robot description, xacro)
@@ -86,10 +86,10 @@
     <!-- VLP-16 -->
     <!--xacro:include filename="$(find velodyne_description)/urdf/VLP-16.urdf.xacro"/>
-    <VLP-16 parent="base_link" name="velodyne" topic="/velodyne_points" hz="10" samples="1024" gpu="true" lasers="32" max_range="50">
-        <origin xyz="0 0 0.2" rpy="0 0 0" />
+    <VLP-16 parent="base_link" name="velodyne" topic="/velodyne_points" hz="10" samples="1024" gpu="true" lasers="16" max_range="50">
+        <origin xyz="0 0 0.3" rpy="0 0 0" />
     </VLP-16-->
     <!-- VHDL-32E -->
 	<xacro:include filename="$(find velodyne_description)/urdf/HDL-32E.urdf.xacro"/>
-  	<HDL-32E parent="base_link" name="velodyne" topic="/velodyne_points" hz="10" samples="1024" gpu="true" lasers="64" max_range="50">
+  	<HDL-32E parent="base_link" name="velodyne" topic="/velodyne_points" hz="10" samples="1024" gpu="true" lasers="32" max_range="50">
     	<origin xyz="0 0 0.4" rpy="0 0 0" />
   	</HDL-32E>
