Commit message: 解决了贴图和方框问题

File: packages/UAV/target_tracking/urdf/scout_v2.xacro (robot description, xacro)
@@ -99,5 +99,5 @@
         <!--origin xyz="0 0 0" rpy="0 0 0" /-->
     </sensor_kinect>
-  <link name="mark_label_1__link">
+  <link name="mark_label_1_link">
     <inertial>
       <mass value="0.390"/>
@@ -105,14 +105,14 @@
       <inertia ixx="0.00058" ixy="0" ixz="0" iyy="0.00058" iyz="0" izz="0.00019"/>
     </inertial>
-    <collision name="mark_label_1__collision">
-      <origin xyz="0 0 1.5707" rpy="0 0 0"/>
+    <collision>
+      <origin xyz="0 0 0.5707" rpy="0 0 0"/>
       <geometry>
-        <box size=".5 .5 .0001"/>
+        <mesh filename="package://target_tracking/models/box_target_green/meshes/mesh.dae" scale="0.2 0.2 0.04"/>
       </geometry>
     </collision>
-    <visual name="mark_label_1__visual">
-      <origin xyz="0 0 1.5707" rpy="0 0 0"/>
+    <visual>
+      <origin xyz="0 0 0.5707" rpy="0 0 0"/>
       <geometry>
-        <box size=".5 .5 .001"/>
+        <mesh filename="package://target_tracking/models/box_target_green/meshes/mesh.dae" scale="0.2 0.2 0.04"/>
       </geometry>
     </visual>
@@ -121,5 +121,5 @@
         <origin xyz="0 0 0" rpy="0 0 0" />
         <parent link="base_link" />
-        <child link="mark_label_1__link" />
+        <child link="mark_label_1_link" />
     </joint>
     <!-- imu link config -->
