Commit message: 简化target_tracking文件目录

File: packages/UAV/target_tracking/models/scout_v2.xacro (robot description, xacro)
@@ -83,5 +83,5 @@
     <xacro:include filename="$(arg urdf_extras)" />
     <!-- Gazebo definitions  -->
-    <xacro:include filename="$(find target_tracking)/urdf/scout_v2.gazebo" />
+    <xacro:include filename="$(find target_tracking)/models/scout_v2.gazebo" />
     <!-- VLP-16 -->
     <!-- <xacro:include filename="$(find velodyne_description)/urdf/VLP-16.urdf.xacro"/>
@@ -95,5 +95,5 @@
   	</HDL-32E>  -->
     <!-- kinect link config -->
-    <xacro:include filename="$(find target_tracking)/urdf/sensors/kinect.urdf.xacro"/>
+    <xacro:include filename="$(find target_tracking)/models/sensors/kinect.urdf.xacro"/>
     <sensor_kinect  parent="base_link">
         <!--origin xyz="0 0 0" rpy="0 0 0" /-->

File: packages/UAV/target_tracking/models/sensors/kinect.urdf.xacro (robot description, xacro)
@@ -1,6 +1,6 @@
 <?xml version="1.0"?>
 <robot name="sensor_kinect" xmlns:xacro="http://ros.org/wiki/xacro">
-  <xacro:include filename="$(find target_tracking)/urdf/sensors/kinect_gazebo.urdf.xacro"/>
-  <xacro:include filename="$(find target_tracking)/urdf/sensors/kinect_properties.urdf.xacro"/>
+  <xacro:include filename="$(find target_tracking)/models/sensors/kinect_gazebo.urdf.xacro"/>
+  <xacro:include filename="$(find target_tracking)/models/sensors/kinect_properties.urdf.xacro"/>
   <xacro:property name="kinect_cam_py" value="-0.0125"/>
   <!-- Parameterised in part by the values in turtlebot_properties.urdf.xacro -->
@@ -28,5 +28,5 @@
         <geometry>
          <!-- <mesh filename="package://turtlebot_description/meshes/sensors/kinect.dae"/> -->
-         <mesh filename="package://target_tracking/meshes/sensors/kinect.dae"/>
+         <mesh filename="package://target_tracking/models/sensors/meshes/sensors/kinect.dae"/>
         </geometry>
       </visual>
