Commit message: update scout_ros

File: packages/UGV/scout_ros/scout_description/urdf/scout_v2.xacro (robot description, xacro)
@@ -6,5 +6,5 @@
     <xacro:include filename="$(find scout_description)/urdf/scout_wheel_type1.xacro" />
     <xacro:include filename="$(find scout_description)/urdf/scout_wheel_type2.xacro" />
-    <xacro:include filename="$(find scout_description)/urdf/sensors/kinect.urdf.xacro"/>
+    <!-- <xacro:include filename="$(find scout_description)/urdf/sensors/kinect.urdf.xacro"/> -->
     <!-- Variables -->
     <xacro:property name="M_PI" value="3.14159"/>
@@ -86,4 +86,26 @@
     <xacro:include filename="$(find scout_description)/urdf/scout_v2.gazebo" />
     <!-- kinect link config -->
-    <sensor_kinect  parent="base_link"/>
+    <!-- <sensor_kinect  parent="base_link"/> -->
+        <!-- VLP-16 -->
+    <!-- <xacro:include filename="$(find velodyne_description)/urdf/VLP-16.urdf.xacro"/> -->
+    <!-- <xacro:VLP-16 parent="base_link" name="velodyne" topic="/velodyne_points" hz="10" samples="1024" gpu="true" lasers="16" max_range="80">
+        <origin xyz="0 0 0.4" rpy="0 0 0" />
+    </xacro:VLP-16> -->
+    <!-- VHDL-32E -->
+    <xacro:include filename="$(find velodyne_description)/urdf/HDL-32E.urdf.xacro"/>
+  	<xacro:HDL-32E parent="base_link" name="velodyne" topic="/velodyne_points" hz="10" samples="1024" gpu="true" lasers="32" max_range="80">
+        <origin xyz="0 0 0.4" rpy="0 0 0" />
+  	</xacro:HDL-32E>
+    <!-- kinect link config -->
+    <xacro:include filename="$(find scout_description)/urdf/sensors/kinect.urdf.xacro"/>
+    <xacro:sensor_kinect parent="base_link">
+        <!--origin xyz="0 0 0" rpy="0 0 0" /-->
+    </xacro:sensor_kinect>
+    <!-- imu link config -->
+    <link name="imu_link" />
+    <joint name="imu_joint" type="fixed">
+        <origin xyz="0 0 0" rpy="0 0 0" />
+        <parent link="base_link" />
+        <child link="imu_link" />
+    </joint>
 </robot>

File: packages/UGV/scout_ros/scout_description/urdf/sensors/kinect.urdf.xacro (robot description, xacro)
@@ -66,5 +66,5 @@
   </joint> -->
 	<!-- Kinect sensor for simulation -->
-	<gazebo_sim_3dsensor/>
+	<xacro:gazebo_sim_3dsensor/>
   </xacro:macro>
 </robot>
